File: pcb/business card.kicad_pcb (KiCad board)
At the start: 2 copper layers, 50 x 82 mm, 289 parts, among them J1 Conn_ST_STDC14, SW1 SW_SPDT, U1 STM32C031G6Ux, U2 TPS61023DRLR, U3 TLV71333PDBV, U4 74AHCT1G125

Commit message: Update PCB design and project overview
Other:
- board text added: "04xxxxxxxx"
- board text added: "xxxxxxxxxxx@hotmail.com"
- board text removed: "0455166930"
- board text removed: "jaxonteague@hotmail.com"
Changed lines of the file:
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@@
 		(capping no)
 		(filling no)
-		(zone_defaults)
 		(pcbplotparams
 			(layerselection 0x00000000_00000000_55555555_5755f5ff)
@@
 				(font
 					(size 1.27 1.27)
+					(thickness 0.15)
 				)
 			)
@@
 		)
 	)
-	(gr_text "0455166930"
+	(gr_text "04xxxxxxxx"
 		(at 16 72.301602 0)
 		(layer "F.SilkS")
@@
 		)
 	)
-	(gr_text "jaxonteague@hotmail.com"
+	(gr_text "xxxxxxxxxxx@hotmail.com"
 		(at 16 76.1 0)
 		(layer "F.SilkS")
